File: adapters/AdapterDIP8M16/AdapterDIP8M16.brd (EAGLE design)
At the start: 59.1 x 62.9 mm, 19 parts, among them M1 ATMEL_MEGA16-P, M4 ATMEL_MEGA8-P

Commit message: t32u4
Other:
- board text added: "GND"
- board text added: "MISO"
- board text added: "MOSI"
- board text added: "RESET"
- board text added: "SCK"
- board text added: "VCC"
Changed lines of the file:
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@@
 <text x="52.07" y="50.27625" size="2.6" layer="1" font="vector" ratio="15" rot="R90.1">e</text>
 <text x="52.07" y="53.45125" size="2.6" layer="1" font="vector" ratio="15" rot="R90.1">M</text>
+<text x="56.1975" y="36.5125" size="1.778" layer="21" font="vector">SCK</text>
+<text x="47.9425" y="42.545" size="1.778" layer="21" font="vector">MISO</text>
+<text x="47.625" y="46.0375" size="1.778" layer="21" font="vector">MOSI</text>
+<text x="37.465" y="38.1" size="1.778" layer="21" font="vector">RESET</text>
+<text x="57.4675" y="20.32" size="1.778" layer="21" font="vector">GND</text>
+<text x="51.435" y="38.4175" size="1.778" layer="21" font="vector" rot="R180">VCC</text>
 </plain>
 <attributes>
@@
 <element name="U$13" library="AdapterDIP8M16" package="PIN" value="PIN" x="51.7525" y="34.29"/>
 <element name="J" library="HWProgUSB" package="RCL_M1206" value="0" x="55.5625" y="34.29" smashed="yes">
-<attribute name="NAME" x="58.7375" y="33.655" size="1.27" layer="25"/>
+<attribute name="NAME" x="55.88" y="31.4325" size="1.27" layer="25"/>
 <attribute name="VALUE" x="54.2925" y="31.75" size="1.27" layer="27"/>
 </element>
