File: adapters/leonardo32u4hvpp/leonardo32u4hvpp.brd (EAGLE design)
At the start: 68.6 x 53.3 mm, 15 parts, among them J2 8x1F-H8.5, J3 8x1F-H8.5, J4 6x1F-H8.5, Y1 16MHz KX-7

Commit message: t32u4
Parts:
- moved U$2 60.3 mm to (113.7, 22.7), turned to 90 degrees
- moved J2 34.8 mm to (82.9, 71.1)
- moved J3 34.8 mm to (65.1, 22.9)
- moved C4 34.8 mm to (76.5, 52.1)
- moved J4 34.8 mm to (85.4, 22.9)
- moved JP1 34.8 mm to (58.5, 71.1)
- moved R1 34.8 mm to (76.5, 45.7)
- moved RESET 34.8 mm to (34.6, 69.7)
- moved RX 34.8 mm to (32.7, 48.3)
- moved RXLED 34.8 mm to (31.6, 48.3)
- moved TX 34.8 mm to (32.7, 44.5)
- moved TXLED 34.8 mm to (31.6, 44.5)
- moved XTAL1 34.8 mm to (75.6, 52.1)
- moved Y1 34.8 mm to (77.2, 48.9)
- moved ICSP 34.8 mm to (93.2, 48.3)
Connections:
- removed net VIN: J3.8
- net +5V: no longer J3.2, J3.5
- net D2/SDA: no longer JP1.9
- net D3/SCL: no longer JP1.10
- net GND: no longer C4.2, J3.6, J3.7, JP1.7, Y1.2, Y1.4
- net RESET: no longer J3.3
Routing:
- net RESET: track 0.00 -> 134.9 mm
- net TXLED: track 0.00 -> 101.1 mm, vias 0 -> 4
- net D0(RXLED): track 0.00 -> 90.9 mm
- net IO12: track 0.00 -> 65.5 mm
- net D5(IO9*): track 20.2 -> 80.3 mm
- net IO10*: track 20.4 -> 80.3 mm
- net XTAL1: track 0.00 -> 59.8 mm, vias 0 -> 2
- net IO11*: track 21.0 -> 79.4 mm, vias 0 -> 2
- net D4(IO8): track 19.7 -> 74.2 mm
- net +5V: track 0.00 -> 49.5 mm, vias 0 -> 2
- net GND: track 124.1 -> 173.3 mm, vias 0 -> 3
- net D6*: track 0.00 -> 45.3 mm, vias 0 -> 2
- net BS2(D7): track 12.3 -> 54.7 mm, vias 1 -> 0
- net D4: track 0.00 -> 42.2 mm
- net D2/SDA: track 0.00 -> 37.7 mm
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Other:
- board size 68.6 x 53.3 mm -> 81.9 x 62.5 mm
- board text removed: "Arduino"
- board text removed: "D.Cuartielles"
- board text removed: "D.Mellis"
- board text removed: "Edition"
- board text removed: "G.Martino"
- board text removed: "LEONARDO"
- board text removed: "Limited"
- board text removed: "M"
- board text removed: "M.Banzi"
- board text removed: "Prototype"
- board text removed: "T.Igoe"
- board text removed: "TM"
- board text removed: "a"
- board text removed: "e"
- board text removed: "g"
- board text removed: "www.arduino.cc"

Commit message: t32u4
Parts:
- added RXLED1, TXLED1: (no value), pinhead:1X01
- moved J2 31.7 mm to (56.2, 54.0)
- moved J3 31.7 mm to (38.4, 5.71)
- moved C4 31.7 mm to (49.8, 34.9)
- moved TX 31.7 mm to (6.03, 27.3)
- moved U$2 31.7 mm to (87.0, 5.56)
- moved Y1 31.7 mm to (50.5, 31.8)
- moved ICSP 31.7 mm to (66.5, 31.1)
- moved J4 31.7 mm to (58.7, 5.71)
- moved JP1 31.7 mm to (31.8, 54.0)
- moved R1 31.7 mm to (49.8, 28.6)
- moved RESET 31.7 mm to (7.94, 52.6)
- moved RX 31.7 mm to (6.03, 31.1)
- moved RXLED 31.7 mm to (4.92, 31.1)
- moved TXLED 31.7 mm to (4.92, 27.3)
- moved XTAL1 31.7 mm to (48.9, 34.9)
Connections:
- net D0(RXLED): now also RXLED1.1
- net TXLED: now also TXLED1.1
Routing:
- net RESET: track 134.9 -> 137.4 mm

Commit message: t32u4
Parts:
- added ICSP_OFF: (no value), SmartPrj:2X03
- added J1: J, detali_main:R1206W
- added JP, RES: (no value), pinhead:1X01
Connections:
- new net N$10: RES.1, U$2.RESET
- new net N$4: J1.2, U$2.D1
- new net N$5: ICSP_OFF.5, U$2.D7
- new net N$6: ICSP_OFF.3, U$2.D6
- new net N$8: ICSP_OFF.1, U$2.D5
- net D1(SCK): now also J1.1; no longer U$2.D1
- net D5(IO9*): now also ICSP_OFF.2; no longer U$2.D5
- net IO10*: now also ICSP_OFF.4; no longer U$2.D6
- net IO11*: now also ICSP_OFF.6; no longer U$2.D7
- net RESET: now also JP.1; no longer U$2.RESET
Routing:
- net D1(SCK): track 44.5 -> 4.05 mm, vias 2 -> 0
- net N$4: track 0.00 -> 34.8 mm
- net RESET: track 137.4 -> 124.2 mm
- net N$10: track 0.00 -> 10.7 mm
- net D5(IO9*): track 80.3 -> 71.4 mm
- net IO11*: track 79.4 -> 70.8 mm
- net IO10*: track 80.3 -> 72.1 mm
- net N$8: track 0.00 -> 6.35 mm
- net N$6: track 0.00 -> 6.35 mm
- net N$5: track 0.00 -> 6.35 mm
- net XTAL1: track 59.8 -> 55.2 mm
- net TXLED: track 101.1 -> 104.9 mm
- net GND: track 173.3 -> 170.4 mm
