File: adapters/AdapterQFP48forZIF/AdapterQFP48forZIF.brd (EAGLE design)
At the start: 54 x 62.9 mm, 15 parts, among them IC1 MEGA8-AI, IC2 MEGA8-P, M4 ATMEL_MEGA8-P

Commit message: 1
Parts:
- removed IC1: MEGA8-AI, atmel:TQFP32-08
- removed IC2: MEGA8-P, atmel:DIL28-3
- removed J: 0, HWProgUSB:RCL_M1206
- removed M4: ATMEL_MEGA8-P, AdapterDIP8M16:ATMEL_DIL28-3
- removed U$10, U$11, U$12, U$13, U$8, U$9: PIN, AdapterDIP8M16:PIN
- added C3: 100n, HWProgUSB:RCL_C0805
- added ISP: (no value), con-lstb:MA03-2
- added J1: 0, rcl:R1206W
- F: value 0 -> 0603
- moved C1 149.1 mm to (45.1, 40.0), flipped to the bottom
- moved C2 138.3 mm to (54.6, 20.0), flipped to the bottom, turned to 90 degrees
- moved U$1 20.3 mm to (14.6, 67.6)
- moved F 17.5 mm to (23.5, 21.3), flipped to the bottom, turned to 90 degrees
- moved U$14 14.5 mm to (49.8, 39.1)
Connections:
- removed net AVCC: IC1.18, IC2.20
- removed net VCC2: C1.1, J.1, U$13.P$1
- new net N$6: ISP.3, J1.2
- net BS1: no longer M4.106
- net BS2: no longer M4.125
- net D0: no longer M4.114
- net D1: no longer M4.115
- net D2: no longer M4.116
- net D3: now also ISP.4; no longer M4.117, U$12.P$1
- net D4: now also ISP.1; no longer M4.118, U$8.P$1
- net D5: now also J1.1; no longer M4.119, U$9.P$1
- net D6: no longer M4.123
- net D7: no longer M4.124
- net GND: now also C3.2, ISP.6; no longer IC1.21, IC1.3, IC1.5, IC2.22, IC2.8, M4.108, M4.122, U$11.P$1
- net OE: no longer M4.104
- net PAGEL: no longer M4.113
- net R/B: no longer M4.103
- net RESET: now also ISP.5; no longer M4.101, U$10.P$1
- net VCC: now also C1.1, C3.1, ISP.2; no longer IC1.4, IC1.6, IC2.7, J.2, M4.107, M4.120
- net WR: no longer M4.105
- net XA0: no longer M4.111
- net XA1: no longer M4.112
- net XTAL1: no longer M4.109
Routing:
- net D6: track 120.5 -> 80.0 mm, vias 3 -> 1
- net GND: track 206.7 -> 171.3 mm, vias 0 -> 2
- net D5: track 125.2 -> 149.8 mm
- net BS2: track 88.2 -> 69.7 mm, vias 3 -> 1
- net R/B: track 92.3 -> 77.6 mm
- net OE: track 76.6 -> 63.4 mm
- net WR: track 52.2 -> 43.3 mm
- net VCC: track 74.6 -> 83.2 mm, vias 1 -> 0
- net BS1: track 50.8 -> 42.5 mm
- net D0: track 72.9 -> 65.3 mm, vias 0 -> 1
- net D1: track 73.5 -> 66.5 mm, vias 0 -> 1
- net PAGEL: track 36.3 -> 29.6 mm
- net XA1: track 36.3 -> 29.6 mm
- net XA0: track 36.3 -> 29.6 mm
- net D2: track 74.4 -> 67.8 mm, vias 0 -> 1
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- added copper zone on layer 1, net N$5
- added copper zone on layer 1, net N$7
Other:
- board size 54 x 62.9 mm -> 54 x 59.7 mm
- board text removed: "1"
- board text removed: "6"
- board text removed: "8"
- board text removed: "GND"
- board text removed: "M"
- board text removed: "MISO"
- board text removed: "MOSI"
- board text removed: "RESET"
- board text removed: "SCK"
- board text removed: "VCC"
- board text removed: "a"
- board text removed: "e"
- board text removed: "g"
