File: adapters/AdapterQFP48forZIF/AdapterQFP48forZIF.sch (EAGLE design)
At the start: 15 parts, among them IC1 MEGA8-AI, IC2 MEGA8-P, M4 ATMEL_MEGA8-P

Commit message: 1
Parts:
- removed IC1: MEGA8-AI, atmel:MEGA8-AI
- removed IC2: MEGA8-P, atmel:MEGA8-P
- removed J: 0, HWProgUSB:RCL_R-EU_M1206
- removed M4: ATMEL_MEGA8-P, AdapterDIP8M16:ATMEL_MEGA8-P
- removed U$10, U$11, U$12, U$13, U$8, U$9: PIN, AdapterDIP8M16:PIN
- added C3: 100n, HWProgUSB:RCL_C-EUC0805
- added ISP: (no value), con-lstb:MA03-2
- added J1: 0, rcl:R-EU_R1206W
- F: value 0 -> 0603
Connections:
- removed net VCC2: C1.1, J.1, U$13.1
- new net N$6: ISP.3, J1.2
- net BS1: no longer M4.PD4(XCK/T0)
- net BS2: no longer M4.PC2(ADC2)
- net D0: no longer M4.PB0(ICP)
- net D1: no longer M4.PB1(OC1A)
- net D2: no longer M4.PB2(SS/OC1B)
- net D3: now also ISP.4; no longer M4.PB3(MOSI/OC2), U$12.1
- net D4: now also ISP.1; no longer M4.PB4(MISO), U$8.1
- net D5: now also J1.1; no longer M4.PB5(SCK), U$9.1
- net D6: no longer M4.PC0(ADC0)
- net D7: no longer M4.PC1(ADC1)
- net GND: now also C3.2, ISP.6; no longer M4.GND, M4.GND@1, U$11.1
- net OE: no longer M4.PD2(INT0)
- net PAGEL: no longer M4.PD7(AIN1)
- net R/B: no longer M4.PD1(TXD)
- net RESET: now also ISP.5; no longer M4.PC6(/RESET), U$10.1
- net VCC: now also C1.1, C3.1, ISP.2; no longer J.2, M4.AVCC, M4.VCC@1
- net WR: no longer M4.PD3(INT1)
- net XA0: no longer M4.PD5(T1)
- net XA1: no longer M4.PD6(AIN0)
- net XTAL1: no longer M4.PB6(XTAL1/TOSC1)
Other:
- note added: "IC51-0324-1498"
- note added: "NO.B003"
- note added: "NO.SA636"
- note added: "QFP32/D32"
- note removed: "ATmega1284"
- note removed: "ATmega16"
- note removed: "ATmega163"
- note removed: "ATmega164"
- note removed: "ATmega168"
- note removed: "ATmega28"
- note removed: "ATmega32"
- note removed: "ATmega323"
- note removed: "ATmega324"
- note removed: "ATmega48"
- note removed: "ATmega644"
- note removed: "ATmega8"
- note removed: "ATmega8535"
- note removed: "ATmega88"
- note removed: "ATtiny11"
- note removed: "ATtiny12"
- note removed: "ATtiny13"
- note removed: "ATtiny15"
- note removed: "ATtiny22"
- note removed: "ATtiny2313"
- note removed: "ATtiny24"
- note removed: "ATtiny25"
- note removed: "ATtiny26"
- note removed: "ATtiny261"
- note removed: "ATtiny44"
- note removed: "ATtiny45"
- note removed: "ATtiny461"
- note removed: "ATtiny84"
- note removed: "ATtiny85"
- note removed: "ISPM16"
- note removed: "ISPM8"
- note removed: "M1"
- note removed: "M2"
- note removed: "M3"
- note removed: "M4"
- note removed: "M5"
- note removed: "M6"
- moved on the sheet: C1, C2, F
