File: adapters/ZIF_QFP48/QFP48forZIF.brd (EAGLE design)
At the start: 54 x 59.7 mm, 8 parts, among them J1 0

Commit message: rename adapter
Routing:
- net BS2: track 69.7 -> 66.8 mm
- net GND: track 171.3 -> 169.0 mm
- net R/B: track 77.6 -> 79.9 mm
- net XTAL1: track 32.1 -> 32.6 mm

Commit message: bak
Routing:
- net RESET: track 83.5 -> 75.9 mm
- net D5: track 149.8 -> 146.8 mm
- net D0: track 65.3 -> 67.9 mm
- net D7: track 93.1 -> 90.9 mm
- net R/B: track 79.9 -> 78.9 mm
- net D1: track 66.5 -> 67.3 mm
