File: adapters/ZIF_QFP32/QFP32forZIF.brd (EAGLE design)
At the start: 54 x 59.7 mm, 8 parts, among them J1 0

Commit message: .
Parts:
- U$14: device AdapterQFP48forZIF:ADAPTERQFP48FORZIF -> QFP32forZIF:ADAPTERQFP48FORZIF
Changed lines of the file:
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@@
 <setting verticaltext="up"/>
 </settings>
-<grid distance="0.05" unitdist="inch" unit="inch" style="lines" multiple="1" display="yes" altdistance="0.025" altunitdist="inch" altunit="inch"/>
+<grid distance="0.05" unitdist="inch" unit="mil" style="lines" multiple="1" display="yes" altdistance="0.025" altunitdist="inch" altunit="inch"/>
 <layers>
 <layer number="1" name="Top" color="4" fill="1" visible="yes" active="yes"/>
@@
 <attribute name="VALUE" x="28.8925" y="21.2725" size="1.27" layer="28" rot="MR90"/>
 </element>
-<element name="U$14" library="AdapterQFP48forZIF" package="ADAPTERQFP48FORZIF" value="SA636-40" x="49.8475" y="39.0525"/>
+<element name="U$14" library="QFP32forZIF" package="ADAPTERQFP48FORZIF" value="SA636-40" x="49.8475" y="39.0525"/>
 <element name="ISP" library="con-lstb" package="MA03-2" value="" x="27.94" y="18.415" smashed="yes" rot="R270">
 <attribute name="NAME" x="26.9875" y="23.876" size="1.27" layer="25" ratio="10"/>
