File: adapters/ZIF_QFP32/QFP32forZIF.sch (EAGLE design)
At the start: 8 parts, among them J1 0

Commit message: .
Parts:
- U$14: device AdapterQFP48forZIF:SA636-40 -> QFP32forZIF:SA636-40
Changed lines of the file:
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@@
 <part name="GND2" library="supply1" deviceset="GND" device=""/>
 <part name="F" library="HWProgUSB" deviceset="RCL_R-EU_" device="M0805" value="0603"/>
-<part name="U$14" library="AdapterQFP48forZIF" deviceset="SA636-40" device=""/>
+<part name="U$14" library="QFP32forZIF" deviceset="SA636-40" device=""/>
 <part name="FRAME1" library="frames" deviceset="DINA4_L" device=""/>
 <part name="ISP" library="con-lstb" deviceset="MA03-2" device=""/>
