File: programmer_dip/HWProgUSB_DIP.brd (EAGLE design)
At the start: 80 x 65.7 mm, 82 parts, among them X2 P_AVR_V

Commit message: .
Parts:
- moved RJ3 5.09 mm to (87.5, 26.5)
Changed lines of the file:
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@@
 <?xml version="1.0" encoding="utf-8"?>
 <!DOCTYPE eagle SYSTEM "eagle.dtd">
-<eagle version="6.3">
+<eagle version="6.4">
 <drawing>
 <settings>
@@
 <wire x1="62.07125" y1="21.43125" x2="62.07125" y2="23.97125" width="0.4064" layer="114"/>
 <hole x="45.085" y="3.175" drill="3.2"/>
-<dimension x1="-9.525" y1="52.07" x2="-10.795" y2="66.04" x3="-12.065" y3="59.055" layer="1" dtype="vertical"/>
+<dimension x1="-9.525" y1="52.07" x2="-10.795" y2="66.04" x3="-12.065" y3="59.055" textsize="3.5" layer="1" dtype="vertical"/>
 <wire x1="79.99" y1="65.71" x2="0" y2="65.71" width="0" layer="20"/>
 <wire x1="80.01" y1="65.71" x2="80.01" y2="52.375" width="0" layer="20"/>
+<dimension x1="0" y1="-0.9525" x2="80.01" y2="-1.5875" x3="40.005" y3="-10.16" textsize="1.778" layer="21" dtype="horizontal"/>
+<dimension x1="83.5025" y1="65.7225" x2="85.09" y2="0" x3="89.8525" y3="32.86125" textsize="1.778" layer="21" dtype="vertical"/>
 </plain>
 <attributes>
@@
 </element>
 <element name="1VD1" library="diode" package="SMB" value="SS12" x="44.1325" y="19.84375"/>
-<element name="RJ3" library="rcl" package="R1206" value="0" x="87.78875" y="31.59125" smashed="yes">
-<attribute name="NAME" x="84.61044375" y="31.850971875" size="1.27" layer="25" rot="R45"/>
-<attribute name="VALUE" x="86.51875" y="29.05125" size="1.27" layer="27"/>
+<element name="RJ3" library="rcl" package="R1206" value="0" x="87.47125" y="26.51125" smashed="yes">
+<attribute name="NAME" x="84.29294375" y="26.770971875" size="1.27" layer="25" rot="R45"/>
+<attribute name="VALUE" x="86.20125" y="23.97125" size="1.27" layer="27"/>
 </element>
 <element name="RJ4" library="rcl" package="R1206" value="0" x="98.26625" y="40.64" smashed="yes">
@@
 <contactref element="1VD1" pad="A"/>
 <contactref element="RJ3" pad="1"/>
-<wire x1="46.3325" y1="19.84375" x2="86.36675" y2="31.59125" width="0" layer="19" extent="1-1"/>
+<wire x1="46.3325" y1="19.84375" x2="86.04925" y2="26.51125" width="0" layer="19" extent="1-1"/>
 </signal>
 <signal name="N$10">
 <contactref element="RJ3" pad="2"/>
 <contactref element="RJ4" pad="1"/>
-<wire x1="89.21075" y1="31.59125" x2="96.84425" y2="40.64" width="0" layer="19" extent="1-1"/>
+<wire x1="88.89325" y1="26.51125" x2="96.84425" y2="40.64" width="0" layer="19" extent="1-1"/>
 </signal>
 <signal name="N$11">
